File: HW/Eagle/DartScorePcb/DartScorePcb.brd (EAGLE design)
At the start: 55 x 55 mm, 21 parts

Commit message: Working pieces
A lot of pieces are now working by themselves but a lot of work remains for the integration of everything.
Parts:
- removed C10: 100nF, SparkFun-Passives:0805
- removed D1, D2, D3, D4, D5: (no value), SparkFun-LED:LED_3MM
- removed DISP1: ATA8041ARBJ, SparkFun-LED:7-SEGMENT-4DIGIT-20MM
- removed R9: 470, SparkFun-Resistors:0805
- removed S1, S2, S3: RESET, SparkFun-Electromechanical:TACTILE-SWITCH-1101NE
- added C2, C3: 100nF, SparkFun-Passives:0805
- added J1: RESET_BUTTON_LIGHT, SparkFun-Connectors:1X02
- added J10: Sensors1, SparkFun-Connectors:1X04
- added J12, J13: CPU_FAN_CONTROL, SparkFun-Connectors:1X02
- added J2: CAM_BUTTON_SWITCH, SparkFun-Connectors:1X02
- added J3: CAM_BUTTON_LIGHT, SparkFun-Connectors:1X02
- added J4: CAL_BUTTON_SWITCH, SparkFun-Connectors:1X02
- added J5: PLAY_BUTTON_SWITCH, SparkFun-Connectors:1X02
- added J6: CAL_BUTTON_LIGHT, SparkFun-Connectors:1X02
- added J7: RESET_BUTTON_SWITCH, SparkFun-Connectors:1X02
- added J8: PLAY_BUTTON_LIGHT, SparkFun-Connectors:1X02
- added J9: FAN_CONTROL, SparkFun-Connectors:1X02
- added R10, R11, R3: 10k, SparkFun-Resistors:0805
- added T1, T2, T3, T4, T5, T6: BSS138, GeekAmmo:SOT23-3
- R1, R6, R7, R8: value 470 -> 10k
- moved R6 74.6 mm to (25.0, 29.0), flipped to the bottom
- moved R8 68.3 mm to (31.0, 20.5), turned to 180 degrees
- moved C11 65.5 mm to (46.5, 19.1), flipped to the bottom
- moved R7 64.1 mm to (22.0, 20.5), turned to 180 degrees
- moved R2 62.9 mm to (3.50, 20.0), turned to 180 degrees
- moved C1 62.8 mm to (8.50, 19.0), flipped to the bottom
- moved R5 57.9 mm to (18.7, 29.2), flipped to the bottom
- moved R1 48.7 mm to (4.00, 29.5), flipped to the bottom
- moved R4 41.7 mm to (8.00, 20.0), turned to 180 degrees
- moved JP2 35.1 mm to (25.6, 14.1)
Connections:
- removed net CS: JP2.24
- removed net GPIO13: JP2.33
- removed net GPIO17: JP2.11
- removed net GPIO19: JP2.35
- removed net GPIO22: JP2.15
- removed net GPIO26: JP2.37
- removed net GPIO27: JP2.13
- removed net GPIO5: JP2.29
- removed net GPIO6: JP2.31
- removed net INT: JP2.22
- removed net N$12: D4.A, R8.1
- removed net N$14: D5.A, R9.1
- removed net N$5: D1.A, R6.1
- removed net RX: JP2.10
- removed net SCK: JP2.23
- removed net SI: JP2.19
- removed net SO: JP2.21
- removed net TX: JP2.8
- new net 12V: J12.2, J13.1, J9.2
- new net GPIO14: C1.1, J2.1, JP2.8, R1.2
- new net GPIO15: JP2.10, R2.2, T2.1
- new net GPIO8: C3.1, J7.1, JP2.24, R6.2
- new net N$1: J9.1, T5.3
- new net N$3: J12.1, T6.3
- new net N$4: J3.1, T2.3
- new net N$6: J6.1, T3.3
- net 5V: now also J1.2, J3.2, J6.2, J8.2
- net GPIO12: now also J10.3; no longer R7.2
- net GPIO16: now also R11.2, T5.1; no longer R1.2
- net GPIO18: now also R8.2, T6.1
- net GPIO20: now also C11.1, J5.1, R5.2; no longer R8.2
- net GPIO21: now also R10.2, T1.1; no longer R9.2
- net GPIO23: now also C2.1, J4.1, R3.2; no longer C11.1, R5.2, S1.2
- net GPIO24: now also T3.1; no longer C1.1, C10.1, R2.2, S2.2, S3.2
- net GPIO7: now also R7.2, T4.1; no longer R6.2
- net N$2: now also J1.1, T1.3; no longer D3.A, R1.1
- net N$8: now also J8.1, T4.3; no longer D2.A, R7.1
- net VDD: now also J10.1, JP2.1, R1.1, R3.1, R6.1; no longer R2.1, R4.1
- net VSS: now also C2.2, C3.2, J10.2, J13.2, J2.2, J4.2, J5.2, J7.2, JP2.20, JP2.39, R10.1, R11.1, R2.1, R4.1, R7.1, R8.1, T1.2, T2.2, T3.2, T4.2, T5.2, T6.2; no longer C10.2, D1.K, D2.K, D3.K, D4.K, D5.K, JP2.30, JP2.34, S1.1, S2.1, S3.1
Routing:
- net VDD: track 0.00 -> 115.7 mm
- net 5V: track 0.00 -> 65.5 mm
- net GPIO20: track 0.00 -> 59.8 mm
- net GPIO14: track 0.00 -> 43.1 mm
- net GPIO21: track 0.00 -> 41.6 mm
- net GPIO23: track 0.00 -> 33.5 mm
- net GPIO18: track 0.00 -> 23.5 mm, vias 0 -> 1
- net GPIO24: track 0.00 -> 22.3 mm
- net GPIO8: track 0.00 -> 20.5 mm
- net GPIO7: track 0.00 -> 17.0 mm
- net GPIO15: track 0.00 -> 16.6 mm
- net GPIO12: track 0.00 -> 15.9 mm
- net GPIO16: track 0.00 -> 15.7 mm
- net 12V: track 0.00 -> 15.0 mm
- net N$4: track 0.00 -> 14.9 mm
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- added copper zone on layer 1, net VSS
- added copper zone on layer 16, net VSS
Other:
- board size 55 x 55 mm -> 51 x 33 mm
- board text added: "+12V"
- board text added: "+5V"
- board text added: "1W"
- board text added: "3.3V"
- board text added: "CAL."
- board text added: "CAM"
- board text added: "DartScore PCB v 1 Design Pär Sundbäck https://github.com/teddycool/DartScore"
- board text added: "FAN1"
- board text added: "FAN2"
- board text added: "GND"
- board text added: "PLAY"
- board text added: "RESET"
