File: HW/Eagle/DartScorePcb/DartScorePcb.sch (EAGLE design)
At the start: 21 parts

Commit message: Working pieces
A lot of pieces are now working by themselves but a lot of work remains for the integration of everything.
Parts:
- removed C10: 100nF, SparkFun-Passives:CAP0805
- removed D1, D2, D3, D4, D5: (no value), SparkFun-LED:LED3MM
- removed DISP1: ATA8041ARBJ, SparkFun-LED:7-SEGMENT-4DIGIT-20MM-RED
- removed R9: 470, SparkFun-Resistors:RESISTOR0805-RES
- removed S1, S2, S3: RESET, SparkFun-Electromechanical:SWITCH-MOMENTARY-2SMD-1101NE
- added C2, C3: 100nF, SparkFun-Passives:CAP0805
- added J1: RESET_BUTTON_LIGHT, SparkFun-Connectors:M02PTH
- added J10: Sensors1, SparkFun-Connectors:M04PTH
- added J12, J13: CPU_FAN_CONTROL, SparkFun-Connectors:M02PTH
- added J2: CAM_BUTTON_SWITCH, SparkFun-Connectors:M02PTH
- added J3: CAM_BUTTON_LIGHT, SparkFun-Connectors:M02PTH
- added J4: CAL_BUTTON_SWITCH, SparkFun-Connectors:M02PTH
- added J5: PLAY_BUTTON_SWITCH, SparkFun-Connectors:M02PTH
- added J6: CAL_BUTTON_LIGHT, SparkFun-Connectors:M02PTH
- added J7: RESET_BUTTON_SWITCH, SparkFun-Connectors:M02PTH
- added J8: PLAY_BUTTON_LIGHT, SparkFun-Connectors:M02PTH
- added J9: FAN_CONTROL, SparkFun-Connectors:M02PTH
- added R10, R11, R3: 10k, SparkFun-Resistors:RESISTOR0805-RES
- added T1, T2, T3, T4, T5, T6: BSS138, GeekAmmo:N-CHANNEL-MOSFET-BSS138
- R1, R6, R7, R8: value 470 -> 10k
Connections:
- removed net CS: JP2.24
- removed net GPIO13: JP2.33
- removed net GPIO17: JP2.11
- removed net GPIO19: JP2.35
- removed net GPIO22: JP2.15
- removed net GPIO26: JP2.37
- removed net GPIO27: JP2.13
- removed net GPIO5: JP2.29
- removed net GPIO6: JP2.31
- removed net INT: JP2.22
- removed net N$12: D4.A, R8.1
- removed net N$14: D5.A, R9.1
- removed net N$5: D1.A, R6.1
- removed net RX: JP2.10
- removed net SCK: JP2.23
- removed net SI: JP2.19
- removed net SO: JP2.21
- removed net TX: JP2.8
- new net 12V: J12.2, J13.1, J9.2
- new net GPIO14: C1.1, J2.1, JP2.8, R1.2
- new net GPIO15: JP2.10, R2.2, T2.G
- new net GPIO8: C3.1, J7.1, JP2.24, R6.2
- new net N$1: J9.1, T5.D
- new net N$3: J12.1, T6.D
- new net N$4: J3.1, T2.D
- new net N$6: J6.1, T3.D
- net 5V: now also J1.2, J3.2, J6.2, J8.2
- net GPIO12: now also J10.3; no longer R7.2
- net GPIO16: now also R11.2, T5.G; no longer R1.2
- net GPIO18: now also R8.2, T6.G
- net GPIO20: now also C11.1, J5.1, R5.2; no longer R8.2
- net GPIO21: now also R10.2, T1.G; no longer R9.2
- net GPIO23: now also C2.1, J4.1, R3.2; no longer C11.1, R5.2, S1.2
- net GPIO24: now also T3.G; no longer C1.1, C10.1, R2.2, S2.2, S3.2
- net GPIO7: now also R7.2, T4.G; no longer R6.2
- net N$2: now also J1.1, T1.D; no longer D3.A, R1.1
- net N$8: now also J8.1, T4.D; no longer D2.A, R7.1
- net VDD: now also J10.1, JP2.1, R1.1, R3.1, R6.1; no longer R2.1, R4.1
- net VSS: now also C2.2, C3.2, J10.2, J13.2, J2.2, J4.2, J5.2, J7.2, JP2.20, JP2.39, R10.1, R11.1, R2.1, R4.1, R7.1, R8.1, T1.S, T2.S, T3.S, T4.S, T5.S, T6.S; no longer C10.2, D1.C, D2.C, D3.C, D4.C, D5.C, JP2.30, JP2.34, S1.1, S2.1, S3.1
Other:
- note added: "Cpu Fan control switch"
- note added: "Enable opencv calibration"
- note added: "Enable view of CAM mounting pattern"
- note added: "Fan control switch"
- note added: "Play reset"
- note removed: "Calibrate"
- note removed: "Reset"
- moved on the sheet: C1, C11, R1, R2, R4, R5, R6, R7, R8
